File: Single saturation module - transformer.kicad_sch (KiCad schematic)
At the start: 38 parts, among them J1 AudioJack2, J3 AudioJack2, U1 NE5532, U2 NE5532, U4 NE5532

Commit message: version 0.3 update
Parts:
- removed R8: 6.8k, symbol Device:R
- added RV3: 10k, symbol Device:R_Potentiometer_Trim
- renumbered R4 to R12, R5 to R9, U2 to U1, U4 to U1, U1 to U2, U4 to U3, U2 to U3
Connections:
- net GND: now also RV3.1, RV3.2
- net at R9.2, U3.2 (-): now also RV3.3
Other:
- note added: "VTL5C3 R13 = 47k Silonex 32SR3 R12 = 470R Handmade Vactrol with 5mm led and LDR = 47k"
- note added: "wet gain compensation"
- note removed: "VTL5C3 R13 = 47k Silonex 32SR3 R12 = 470R Experiment with handmade vactrols"

Commit message: version 0.3 readme update
Parts:
- removed R?: 100k, symbol Device:R
- added R2: 10k, symbol Device:R
Connections:
- net Audio_in: now also U?.3 (+), R2.1
- net GND: now also R2.2
Changed lines of the file:
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@@
   (junction (at 82.55 110.49) (diameter 0) (color 0 0 0 0)
   )
+  (junction (at 55.88 38.1) (diameter 0) (color 0 0 0 0)
+  )
   (junction (at 133.35 127) (diameter 0) (color 0 0 0 0)
   )
@@
     (stroke (width 0) (type default))
   )
+  (wire (pts (xy 55.88 38.1) (xy 63.5 38.1))
+    (stroke (width 0) (type default))
+  )
   (wire (pts (xy 130.81 92.71) (xy 128.27 92.71))
     (stroke (width 0) (type default))
@@
     (stroke (width 0) (type default))
   )
-  (wire (pts (xy 60.96 38.1) (xy 63.5 38.1))
+  (wire (pts (xy 50.8 38.1) (xy 55.88 38.1))
     (stroke (width 0) (type default))
   )
@@
   )
   (wire (pts (xy 233.68 119.38) (xy 233.68 130.81))
-    (stroke (width 0) (type default))
-  )
-  (wire (pts (xy 50.8 38.1) (xy 53.34 38.1))
     (stroke (width 0) (type default))
   )
@@
         (path "/ec237045-c42e-41b5-9862-2d4c3f861897"
           (reference "Q1") (unit 1)
+        )
+      )
+    )
+  )
+  (symbol (lib_id "power:GND") (at 55.88 45.72 0) (unit 1)
+    (in_bom yes) (on_board yes) (dnp no) (fields_autoplaced)
+    (property "Reference" "#PWR020" (at 55.88 52.07 0)
+      (effects (font (size 1.27 1.27)) hide)
+    )
+    (property "Value" "GND" (at 55.88 50.8 0)
+      (effects (font (size 1.27 1.27)))
+    )
+    (property "Footprint" "" (at 55.88 45.72 0)
+      (effects (font (size 1.27 1.27)) hide)
+    )
+    (property "Datasheet" "" (at 55.88 45.72 0)
+      (effects (font (size 1.27 1.27)) hide)
+    )
+    (pin "1")
+    (instances
+      (project "Single saturation module - transformer"
+        (path "/ec237045-c42e-41b5-9862-2d4c3f861897"
+          (reference "#PWR020") (unit 1)
         )
       )
@@
     )
   )
+  (symbol (lib_id "Device:R") (at 55.88 41.91 0) (unit 1)
+    (in_bom yes) (on_board yes) (dnp no) (fields_autoplaced)
+    (property "Reference" "R2" (at 58.42 40.64 0)
+      (effects (font (size 1.27 1.27)) (justify left))
+    )
+    (property "Value" "10k" (at 58.42 43.18 0)
+      (effects (font (size 1.27 1.27)) (justify left))
+    )
+    (property "Footprint" "" (at 54.102 41.91 90)
+      (effects (font (size 1.27 1.27)) hide)
+    )
+    (property "Datasheet" "~" (at 55.88 41.91 0)
+      (effects (font (size 1.27 1.27)) hide)
+    )
+    (pin "1")
+    (pin "2")
+    (instances
+      (project "Single saturation module - transformer"
+        (path "/ec237045-c42e-41b5-9862-2d4c3f861897"
+          (reference "R2") (unit 1)
+        )
+      )
+    )
+  )
   (symbol (lib_id "power:+12V") (at 180.34 96.52 0) (unit 1)
     (in_bom yes) (on_board yes) (dnp no) (fields_autoplaced)
@@
         )
       )
-    )
-  )
-  (symbol (lib_id "Device:R") (at 57.15 38.1 90) (unit 1)
-    (in_bom yes) (on_board yes) (dnp no) (fields_autoplaced)
-    (property "Reference" "R?" (at 57.15 31.75 90)
-      (effects (font (size 1.27 1.27)))
-    )
-    (property "Value" "100k" (at 57.15 34.29 90)
-      (effects (font (size 1.27 1.27)))
-    )
-    (property "Footprint" "" (at 57.15 39.878 90)
-      (effects (font (size 1.27 1.27)) hide)
-    )
-    (property "Datasheet" "~" (at 57.15 38.1 0)
-      (effects (font (size 1.27 1.27)) hide)
-    )
-    (pin "1")
-    (pin "2")
-    (instances
-      (project "Multi Saturation Module"
-        (path "/8a579165-884d-4b7e-ba97-82c46eacec16"
-          (reference "R?") (unit 1)
-        )
-      )
-      (project "Single saturation module - transformer"
-        (path "/ec237045-c42e-41b5-9862-2d4c3f861897"
-          (reference "R2") (unit 1)
-        )
-      )
