File: Multi_Saturation_Board_A.kicad_sch (KiCad schematic)
At the start: 46 parts, among them J6 EURO_PWR_2x5, J7 EuroPower_JST_3P, J8 Board_A_1, J9 Board_A_2, U1 NE5532, U2 NE5532, U3 VTL5C, U4 NE5532, U5 NE5532

Commit message: board update
Connections:
- net +12V_IN: now reaches D7.2 (A), J6.1 (+12V), J6.2 (+12V), J7.1 (+12v)
- net -12V_IN: now reaches D8.1 (K), J6.10 (-12V), J6.9 (-12V), J7.3 (-12v)
Changed lines of the file:
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@@
     (effects (font (size 1 1)) (justify left bottom))
+  )
+  (label "GND_IN" (at 34.925 178.435 0) (fields_autoplaced)
+    (effects (font (size 1.27 1.27)) (justify left bottom))
+  )
+  (label "+12V_IN" (at 34.29 170.815 0) (fields_autoplaced)
+    (effects (font (size 1.27 1.27)) (justify left bottom))
+  )
+  (label "-12V_IN" (at 33.02 186.055 0) (fields_autoplaced)
+    (effects (font (size 1.27 1.27)) (justify left bottom))
   )
   (global_label "Audio_in" (shape output) (at 229.235 133.985 0) (fields_autoplaced)
@@
   )
   (symbol (lib_id "power:GND") (at 38.1 178.435 0) (unit 1)
-    (in_bom yes) (on_board yes) (dnp no) (fields_autoplaced)
+    (in_bom yes) (on_board yes) (dnp no)
     (property "Reference" "#PWR026" (at 38.1 184.785 0)
       (effects (font (size 1.27 1.27)) hide)
     )
-    (property "Value" "GND" (at 38.1 183.515 0)
-      (effects (font (size 1.27 1.27)))
-    )
+    (property "Value" "GND" (at 38.1 182.245 0)
+      (effects (font (size 1.27 1.27)))
+    )

Commit message: All boards routed
Parts:
- C4, C5: footprint DIYSynthMNL:CP_Radial_D4.0mm_P1.50mm -> Capacitor_THT:CP_Radial_D5.0mm_P2.50mm
Changed lines of the file:
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@@
       (effects (font (size 1.27 1.27)) (justify left))
     )
-    (property "Footprint" "DIYSynthMNL:CP_Radial_D4.0mm_P1.50mm" (at 86.6902 186.055 0)
+    (property "Footprint" "Capacitor_THT:CP_Radial_D5.0mm_P2.50mm" (at 86.6902 186.055 0)
       (effects (font (size 1.27 1.27)) hide)
     )
@@
       (effects (font (size 1.27 1.27)) (justify left))
     )
-    (property "Footprint" "DIYSynthMNL:CP_Radial_D4.0mm_P1.50mm" (at 86.6902 178.435 0)
-      (effects (font (size 1.27 1.27)) hide)
-    )
+    (property "Footprint" "Capacitor_THT:CP_Radial_D5.0mm_P2.50mm" (at 86.6902 178.435 0)
+      (effects (font (size 1.27 1.27)) hide)
+    )

Commit message: board update
Parts:
- J6: value EURO_PWR_2x5 -> EURO_PWR_16P; footprint DIYSynthMNL:IDC-Header_2x05_P2.54mm_Vertical_BigPads -> DIYSynthMNL:IDC-Header_2x08_P2.54mm_Vertical; symbol eurocad:EURO_PWR_2x5 -> DIYSynthMNL:EURO_PWR_16_PIN
Connections:
- net +12V_IN: now also J6.10 (+12V), J6.9 (+12V); no longer J6.1 (+12V), J6.2 (+12V)
- net -12V_IN: now also J6.1 (-12V), J6.2 (-12V); no longer J6.10 (-12V), J6.9 (-12V)
- no-connect marks 3 -> 9
Changed lines of the file:
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@@
   (junction (at 231.14 59.055) (diameter 0) (color 0 0 0 0)
   )
+  (junction (at 70.485 170.815) (diameter 0) (color 0 0 0 0)
+  )
   (junction (at 241.3 59.055) (diameter 0) (color 0 0 0 0)
   )
@@
   (junction (at 81.28 116.205) (diameter 0) (color 0 0 0 0)
   )
+  (junction (at 40.005 173.355) (diameter 0) (color 0 0 0 0)
+  )
   (junction (at 151.765 165.735) (diameter 0) (color 0 0 0 0)
   )
@@
   (junction (at 121.285 170.815) (diameter 0) (color 0 0 0 0)
   )
-  (junction (at 66.04 170.815) (diameter 0) (color 0 0 0 0)
-  )
   (junction (at 83.185 170.815) (diameter 0) (color 0 0 0 0)
   )
   (junction (at 82.55 186.055) (diameter 0) (color 0 0 0 0)
   )
+  (junction (at 69.215 173.355) (diameter 0) (color 0 0 0 0)
+  )
   (junction (at 131.445 170.815) (diameter 0) (color 0 0 0 0)
   )
   (junction (at 137.16 111.125) (diameter 0) (color 0 0 0 0)
   )
-  (junction (at 43.18 170.815) (diameter 0) (color 0 0 0 0)
-  )
   (junction (at 234.95 85.725) (diameter 0) (color 0 0 0 0)
   )
@@
   )
   (no_connect (at 203.2 126.365))
+  (no_connect (at 66.04 165.735))
+  (no_connect (at 43.18 170.815))
   (no_connect (at 93.98 42.545))
+  (no_connect (at 43.18 168.275))
+  (no_connect (at 66.04 168.275))
   (no_connect (at 104.14 42.545))
+  (no_connect (at 66.04 170.815))
+  (no_connect (at 43.18 165.735))
   (wire (pts (xy 231.14 62.865) (xy 231.14 59.055))
     (stroke (width 0) (type default))
@@
     (stroke (width 0) (type default))
   )
+  (wire (pts (xy 66.04 173.355) (xy 69.215 173.355))
+    (stroke (width 0) (type default))
+  )
   (wire (pts (xy 137.16 111.125) (xy 140.97 111.125))
     (stroke (width 0) (type default))
@@
     (stroke (width 0) (type default))
   )
+  (wire (pts (xy 70.485 170.815) (xy 70.485 173.355))
+    (stroke (width 0) (type default))
+  )
   (wire (pts (xy 158.75 41.275) (xy 158.75 48.895))
     (stroke (width 0) (type default))
@@
     (stroke (width 0) (type default))
   )
+  (wire (pts (xy 69.215 163.195) (xy 69.215 173.355))
+    (stroke (width 0) (type default))
+  )
   (wire (pts (xy 44.45 42.545) (xy 43.18 42.545))
     (stroke (width 0) (type default))
@@
     (stroke (width 0) (type default))
   )
-  (wire (pts (xy 66.04 170.815) (xy 43.18 170.815))
+  (wire (pts (xy 229.235 146.685) (xy 229.235 149.225))
     (stroke (width 0) (type default))
   )
-  (wire (pts (xy 229.235 146.685) (xy 229.235 149.225))
+  (wire (pts (xy 69.215 173.355) (xy 70.485 173.355))
     (stroke (width 0) (type default))
   )
@@
     (stroke (width 0) (type default))
   )
+  (wire (pts (xy 70.485 170.815) (xy 72.39 170.815))
+    (stroke (width 0) (type default))
+  )
+  (wire (pts (xy 40.005 163.195) (xy 69.215 163.195))
+    (stroke (width 0) (type default))
+  )
   (wire (pts (xy 85.725 170.815) (xy 111.125 170.815))
     (stroke (width 0) (type default))
@@
     (stroke (width 0) (type default))
   )
-  (wire (pts (xy 66.04 170.815) (xy 72.39 170.815))
-    (stroke (width 0) (type default))
-  )
   (wire (pts (xy 113.03 186.055) (xy 113.03 189.865))
     (stroke (width 0) (type default))
@@
     (stroke (width 0) (type default))
   )
-  (wire (pts (xy 33.02 175.895) (xy 33.02 170.815))
+  (wire (pts (xy 33.02 175.895) (xy 33.02 173.355))
     (stroke (width 0) (type default))
   )
@@
     (stroke (width 0) (type default))
   )
-  (wire (pts (xy 66.04 173.355) (xy 66.04 170.815))
-    (stroke (width 0) (type default))
-  )
   (wire (pts (xy 219.71 61.595) (xy 219.71 59.055))
     (stroke (width 0) (type default))
@@
     (stroke (width 0) (type default))
   )
+  (wire (pts (xy 33.02 173.355) (xy 40.005 173.355))
+    (stroke (width 0) (type default))
+  )
   (wire (pts (xy 137.16 111.125) (xy 137.16 115.57))
     (stroke (width 0) (type default))
@@
     (stroke (width 0) (type default))
   )
-  (wire (pts (xy 43.18 170.815) (xy 43.18 173.355))
-    (stroke (width 0) (type default))
-  )
   (wire (pts (xy 203.2 118.745) (xy 203.2 121.285))
     (stroke (width 0) (type default))
@@
     (stroke (width 0) (type default))
   )
+  (wire (pts (xy 40.005 173.355) (xy 43.18 173.355))
+    (stroke (width 0) (type default))
+  )
   (wire (pts (xy 139.7 38.735) (xy 143.51 38.735))
     (stroke (width 0) (type default))
   )
+  (wire (pts (xy 70.485 167.64) (xy 70.485 170.815))
+    (stroke (width 0) (type default))
+  )
   (wire (pts (xy 189.23 56.515) (xy 204.47 56.515))
     (stroke (width 0) (type default))
@@
     (stroke (width 0) (type default))
   )
-  (wire (pts (xy 33.02 170.815) (xy 43.18 170.815))
+  (wire (pts (xy 40.005 173.355) (xy 40.005 163.195))
     (stroke (width 0) (type default))
   )
@@
     (effects (font (size 1.27 1.27)) (justify left bottom))
   )
-  (label "+12V_IN" (at 34.29 170.815 0) (fields_autoplaced)
+  (label "+12V_IN" (at 34.29 173.355 0) (fields_autoplaced)
     (effects (font (size 1.27 1.27)) (justify left bottom))
   )
@@
     )
   )
-  (symbol (lib_id "power:PWR_FLAG") (at 66.04 170.815 0) (unit 1)
+  (symbol (lib_id "power:PWR_FLAG") (at 70.485 167.64 0) (unit 1)
     (in_bom yes) (on_board yes) (dnp no)
-    (property "Reference" "#FLG?" (at 66.04 168.91 0)
+    (property "Reference" "#FLG?" (at 70.485 165.735 0)
       (effects (font (size 1.27 1.27)) hide)
     )
-    (property "Value" "PWR_FLAG" (at 66.04 165.735 0)
+    (property "Value" "PWR_FLAG" (at 70.485 162.56 0)
       (effects (font (size 1.27 1.27)))
     )
-    (property "Footprint" "" (at 66.04 170.815 0)
+    (property "Footprint" "" (at 70.485 167.64 0)
       (effects (font (size 1.27 1.27)) hide)
     )
-    (property "Datasheet" "~" (at 66.04 170.815 0)
+    (property "Datasheet" "~" (at 70.485 167.64 0)
       (effects (font (size 1.27 1.27)) hide)
     )
@@
     )
   )
-  (symbol (lib_id "eurocad:EURO_PWR_2x5") (at 54.61 178.435 0) (unit 1)
+  (symbol (lib_id "DIYSynthMNL:EURO_PWR_16_PIN") (at 54.61 178.435 0) (unit 1)
     (in_bom yes) (on_board yes) (dnp no)
-    (property "Reference" "J6" (at 54.61 167.005 0)
+    (property "Reference" "J6" (at 54.61 187.325 0)
       (effects (font (size 1.524 1.524)))
     )
-    (property "Value" "EURO_PWR_2x5" (at 54.61 169.545 0)
+    (property "Value" "EURO_PWR_16P" (at 54.61 161.925 0)
       (effects (font (size 1.524 1.524)))
     )
-    (property "Footprint" "DIYSynthMNL:IDC-Header_2x05_P2.54mm_Vertical_BigPads" (at 53.34 189.865 0)
+    (property "Footprint" "DIYSynthMNL:IDC-Header_2x08_P2.54mm_Vertical" (at 48.895 192.405 0)
       (effects (font (size 1.524 1.524)) hide)
     )
@@
     (pin "7")
     (pin "9")
+    (pin "13")
+    (pin "16")
+    (pin "11")
+    (pin "12")
+    (pin "15")
+    (pin "14")
     (instances
       (project "Multi saturation module"

Commit message: cleaned up project directory
Other:
- note added: "Global label format: Reference_Pin_Board"
- note removed: "dry gain compensation"
- note removed: "wet gain compensation"
Changed lines of the file:
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@@
   (title_block
     (title "Eurorack Multi Saturation Module Board A")
-    (date "2023-12-24")
-    (rev "0.5")
+    (date "2023-12-28")
+    (rev "0.6")
     (company "DIYSynthManila")
     (comment 1 "This version is a prototype.")
@@
     (stroke (width 0) (type default))
   )
-  (wire (pts (xy 114.3 108.585) (xy 111.76 108.585))
+  (wire (pts (xy 114.3 112.395) (xy 118.745 112.395))
     (stroke (width 0) (type default))
   )
@@
     (stroke (width 0) (type default))
   )
-  (wire (pts (xy 114.3 104.775) (xy 114.3 108.585))
+  (wire (pts (xy 114.3 104.775) (xy 114.3 112.395))
     (stroke (width 0) (type default))
   )
@@
     (stroke (width 0) (type default))
   )
+  (wire (pts (xy 115.57 121.92) (xy 118.11 121.92))
+    (stroke (width 0) (type default))
+  )
   (wire (pts (xy 85.725 170.815) (xy 111.125 170.815))
     (stroke (width 0) (type default))
@@
     (stroke (width 0) (type default))
   )
-  (wire (pts (xy 109.22 127.635) (xy 109.22 126.365))
-    (stroke (width 0) (type default))
-  )
-  (wire (pts (xy 107.95 126.365) (xy 109.22 126.365))
+  (wire (pts (xy 118.11 124.46) (xy 118.11 121.92))
     (stroke (width 0) (type default))
   )
@@
     (stroke (width 0) (type default))
   )
-  (wire (pts (xy 109.22 127.635) (xy 114.3 127.635))
+  (wire (pts (xy 118.11 124.46) (xy 114.3 124.46))
     (stroke (width 0) (type default))
   )
@@
     (stroke (width 0) (type default))
   )
-  (wire (pts (xy 43.18 118.745) (xy 48.895 118.745))
+  (wire (pts (xy 114.3 124.46) (xy 114.3 127.635))
+    (stroke (width 0) (type default))
+  )
+  (wire (pts (xy 43.18 118.745) (xy 46.355 118.745))
     (stroke (width 0) (type default))
   )
@@
     (effects (font (size 1.27 1.27)) (justify left bottom))
   )
-  (text "dry gain compensation\n" (at 132.08 127.635 0)
-    (effects (font (size 1 1)) (justify left bottom))
-  )
   (text "Input buffer" (at 33.02 27.305 0)
     (effects (font (size 1.27 1.27)) (justify left bottom))
@@
     (effects (font (size 1.27 1.27)) (justify left bottom))
   )
-  (text "Op Amp bypass caps" (at 124.46 156.21 0)
-    (effects (font (size 1.27 1.27)) (justify left bottom))
-  )
-  (text "wet gain compensation\n" (at 92.71 104.775 0)
-    (effects (font (size 1 1)) (justify left bottom))
+  (text "Op Amp bypass caps" (at 126.365 156.21 0)
+    (effects (font (size 1.27 1.27)) (justify left bottom))
+  )
+  (text "Global label format: Reference_Pin_Board" (at 189.865 158.115 0)
+    (effects (font (size 1.27 1.27)) (justify left bottom))
   )
   (label "GND_IN" (at 34.925 178.435 0) (fields_autoplaced)
@@
     )
   )
-  (global_label "RV4_3" (shape passive) (at 48.895 118.745 0) (fields_autoplaced)
-    (effects (font (size 1.27 1.27)) (justify left))
-    (property "Intersheetrefs" "${INTERSHEET_REFS}" (at 56.5141 118.745 0)
+  (global_label "RV4_3" (shape passive) (at 46.355 118.745 0) (fields_autoplaced)
+    (effects (font (size 1.27 1.27)) (justify left))
+    (property "Intersheetrefs" "${INTERSHEET_REFS}" (at 53.9741 118.745 0)
       (effects (font (size 1.27 1.27)) (justify left) hide)
     )
@@
     )
   )
-  (global_label "RV2_3" (shape passive) (at 111.76 108.585 180) (fields_autoplaced)
-    (effects (font (size 1.27 1.27)) (justify right))
-    (property "Intersheetrefs" "${INTERSHEET_REFS}" (at 104.1409 108.585 0)
-      (effects (font (size 1.27 1.27)) (justify right) hide)
+  (global_label "RV2_3" (shape passive) (at 118.745 112.395 0) (fields_autoplaced)
+    (effects (font (size 1.27 1.27)) (justify left))
+    (property "Intersheetrefs" "${INTERSHEET_REFS}" (at 126.3641 112.395 0)
+      (effects (font (size 1.27 1.27)) (justify left) hide)
     )
   )
@@
     )
   )
-  (global_label "D4_-" (shape passive) (at 107.95 126.365 180) (fields_autoplaced)
-    (effects (font (size 1.27 1.27)) (justify right))
-    (property "Intersheetrefs" "${INTERSHEET_REFS}" (at 101.0566 126.365 0)
-      (effects (font (size 1.27 1.27)) (justify right) hide)
-    )
+  (global_label "D4_-" (shape passive) (at 115.57 121.92 180) (fields_autoplaced)
+    (effects (font (size 1.27 1.27)) (justify right))
+    (property "Intersheetrefs" "${INTERSHEET_REFS}" (at 108.6766 121.92 0)
+      (effects (font (size 1.27 1.27)) (justify right) hide)
+    )

Commit message: board and schematic update
Parts:
- added H1, H2: MountingHole, DIYSynthMNL:MountingHole_M3_Standoff_Pad, symbol Mechanical:MountingHole_Pad
Connections:
- net GND: now also H1.1, H2.1
Changed lines of the file:
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@@
   (junction (at 85.725 178.435) (diameter 0) (color 0 0 0 0)
+  )
+  (junction (at 260.985 126.365) (diameter 0) (color 0 0 0 0)
   )
   (junction (at 43.18 178.435) (diameter 0) (color 0 0 0 0)
@@
     (stroke (width 0) (type default))
   )
+  (wire (pts (xy 260.985 126.365) (xy 260.985 119.38))
+    (stroke (width 0) (type default))
+  )
   (wire (pts (xy 33.02 180.975) (xy 33.02 186.055))
     (stroke (width 0) (type default))
@@
     (stroke (width 0) (type default))
   )
+  (wire (pts (xy 260.985 126.365) (xy 265.43 126.365))
+    (stroke (width 0) (type default))
+  )
   (wire (pts (xy 80.01 186.055) (xy 82.55 186.055))
     (stroke (width 0) (type default))
@@
   )
   (wire (pts (xy 81.28 116.205) (xy 90.17 116.205))
+    (stroke (width 0) (type default))
+  )
+  (wire (pts (xy 260.985 119.38) (xy 265.43 119.38))
     (stroke (width 0) (type default))
   )
@@
     )
   )
+  (symbol (lib_id "power:GND") (at 260.985 126.365 0) (unit 1)
+    (in_bom yes) (on_board yes) (dnp no) (fields_autoplaced)
+    (property "Reference" "#PWR032" (at 260.985 132.715 0)
+      (effects (font (size 1.27 1.27)) hide)
+    )
+    (property "Value" "GND" (at 260.985 130.81 0)
+      (effects (font (size 1.27 1.27)))
+    )
+    (property "Footprint" "" (at 260.985 126.365 0)
+      (effects (font (size 1.27 1.27)) hide)
+    )
+    (property "Datasheet" "" (at 260.985 126.365 0)
+      (effects (font (size 1.27 1.27)) hide)
+    )
+    (pin "1")
+    (instances
+      (project "Multi saturation module"
+        (path "/ec237045-c42e-41b5-9862-2d4c3f861897/c30b6378-be73-4bdd-8ae7-082c1f6babb1"
+          (reference "#PWR032") (unit 1)
+        )
+        (path "/ec237045-c42e-41b5-9862-2d4c3f861897/3a05c5ff-a267-4ce4-8e92-6d5107775c32"
+          (reference "#PWR037") (unit 1)
+        )
+      )
+    )
+  )
   (symbol (lib_id "Device:R") (at 215.9 48.895 90) (unit 1)
     (in_bom yes) (on_board yes) (dnp no) (fields_autoplaced)
@@
         (path "/ec237045-c42e-41b5-9862-2d4c3f861897/3a05c5ff-a267-4ce4-8e92-6d5107775c32"
           (reference "R21") (unit 1)
+        )
+      )
+    )
+  )
+  (symbol (lib_id "Mechanical:MountingHole_Pad") (at 265.43 123.825 0) (unit 1)
+    (in_bom yes) (on_board yes) (dnp no) (fields_autoplaced)
+    (property "Reference" "H2" (at 268.605 121.285 0)
+      (effects (font (size 1.27 1.27)) (justify left))
+    )
+    (property "Value" "MountingHole" (at 268.605 123.825 0)
+      (effects (font (size 1.27 1.27)) (justify left))
+    )
+    (property "Footprint" "DIYSynthMNL:MountingHole_M3_Standoff_Pad" (at 265.43 123.825 0)
+      (effects (font (size 1.27 1.27)) hide)
+    )
+    (property "Datasheet" "~" (at 265.43 123.825 0)
+      (effects (font (size 1.27 1.27)) hide)
+    )
+    (pin "1")
+    (instances
+      (project "Multi saturation module"
+        (path "/ec237045-c42e-41b5-9862-2d4c3f861897/c30b6378-be73-4bdd-8ae7-082c1f6babb1"
+          (reference "H2") (unit 1)
+        )
+        (path "/ec237045-c42e-41b5-9862-2d4c3f861897/3a05c5ff-a267-4ce4-8e92-6d5107775c32"
+          (reference "H2") (unit 1)
         )
       )
@@
         )
       )
+    )
+  )
+  (symbol (lib_id "Mechanical:MountingHole_Pad") (at 265.43 116.84 0) (unit 1)
+    (in_bom yes) (on_board yes) (dnp no) (fields_autoplaced)
+    (property "Reference" "H1" (at 268.605 114.3 0)
+      (effects (font (size 1.27 1.27)) (justify left))
+    )
+    (property "Value" "MountingHole" (at 268.605 116.84 0)
+      (effects (font (size 1.27 1.27)) (justify left))
+    )
+    (property "Footprint" "DIYSynthMNL:MountingHole_M3_Standoff_Pad" (at 265.43 116.84 0)
+      (effects (font (size 1.27 1.27)) hide)
+    )
+    (property "Datasheet" "~" (at 265.43 116.84 0)
+      (effects (font (size 1.27 1.27)) hide)
+    )
+    (pin "1")
+    (instances
+      (project "Multi saturation module"
+        (path "/ec237045-c42e-41b5-9862-2d4c3f861897/c30b6378-be73-4bdd-8ae7-082c1f6babb1"
+          (reference "H1") (unit 1)
+        )
+        (path "/ec237045-c42e-41b5-9862-2d4c3f861897/3a05c5ff-a267-4ce4-8e92-6d5107775c32"
+          (reference "H1") (unit 1)
+        )
+      )
