File: Multi_Saturation_Board_B.kicad_sch (KiCad schematic)
At the start: 21 parts, among them J1 Audio_in, J3 Mix_audio_out, J5 Wet_audio_out, J8 Board_B_1, J9 Board_B_2, SW2 Opto_bypass, SW3 Clipping

Commit message: All boards routed
Connections:
- net +12V renamed +12VA
- net -12V renamed -12VA
- net Audio_in renamed Audio_in_B
- net Clipping_diodes renamed Clipping_diodes_B
- net D1_+ renamed D1_+_B
- net D1_- renamed D1_-_B
- net D4_+ renamed D4_+_B
- net D4_- renamed D4_-_B
- net GND renamed GND1
- net Mix_CV_in renamed Mix_CV_in_B
- net Mix_audio_out renamed Mix_audio_out_B
- net RV1_2 renamed RV1_2_B
- net RV2_3 renamed RV2_3_B
- net RV3_3 renamed RV3_3_B
- net RV4_2 renamed RV4_2_B
- net RV4_3 renamed RV4_3_B
- net SW1_1 renamed SW1_1_B
- net SW1_2 renamed SW1_2_B
- net SW1_4 renamed SW1_4_B
- net SW1_5 renamed SW1_5_B
- net SW2_1 renamed SW2_1_B
- net SW2_2 renamed SW2_2_B
- net SW2_4 renamed SW2_4_B
- net SW2_5 renamed SW2_5_B
- net Wet renamed Wet_B

Commit message: board update
Parts:
- J8, J9: footprint Connector_PinHeader_2.54mm:PinHeader_1x16_P2.54mm_Vertical -> Connector_PinSocket_2.54mm:PinSocket_1x16_P2.54mm_Vertical
Changed lines of the file:
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@@
     (comment 1 "This version is a prototype.")
   )
+  (junction (at 37.465 153.035) (diameter 0) (color 0 0 0 0)
+  )
   (junction (at 69.215 184.15) (diameter 0) (color 0 0 0 0)
   )
   (junction (at 37.465 154.305) (diameter 0) (color 0 0 0 0)
   )
+  (junction (at 37.465 149.225) (diameter 0) (color 0 0 0 0)
+  )
   (junction (at 70.485 82.55) (diameter 0) (color 0 0 0 0)
   )
@@
   )
   (junction (at 74.295 92.71) (diameter 0) (color 0 0 0 0)
+  )
+  (junction (at 37.465 159.385) (diameter 0) (color 0 0 0 0)
   )
   (junction (at 66.675 92.71) (diameter 0) (color 0 0 0 0)
@@
     (stroke (width 0) (type default))
   )
-  (wire (pts (xy 37.465 151.765) (xy 37.465 154.305))
+  (wire (pts (xy 37.465 151.765) (xy 37.465 153.035))
     (stroke (width 0) (type default))
   )
@@
     (stroke (width 0) (type default))
   )
+  (wire (pts (xy 37.465 157.48) (xy 23.495 157.48))
+    (stroke (width 0) (type default))
+  )
   (wire (pts (xy 74.295 82.55) (xy 74.295 83.82))
     (stroke (width 0) (type default))
@@
     (stroke (width 0) (type default))
   )
+  (wire (pts (xy 23.495 153.035) (xy 37.465 153.035))
+    (stroke (width 0) (type default))
+  )
   (wire (pts (xy 69.215 179.07) (xy 69.215 181.61))
     (stroke (width 0) (type default))
@@
     (stroke (width 0) (type default))
   )
+  (wire (pts (xy 23.495 153.035) (xy 23.495 153.67))
+    (stroke (width 0) (type default))
+  )
   (wire (pts (xy 145.415 70.485) (xy 142.875 70.485))
     (stroke (width 0) (type default))
   )
+  (wire (pts (xy 37.465 153.035) (xy 37.465 154.305))
+    (stroke (width 0) (type default))
+  )
   (wire (pts (xy 146.685 78.105) (xy 146.685 81.915))
     (stroke (width 0) (type default))
@@
   )
   (wire (pts (xy 67.945 62.23) (xy 70.485 62.23))
+    (stroke (width 0) (type default))
+  )
+  (wire (pts (xy 37.465 157.48) (xy 37.465 159.385))
     (stroke (width 0) (type default))
   )
@@
       (effects (font (size 1.27 1.27)) (justify left))
     )
-    (property "Footprint" "Connector_PinHeader_2.54mm:PinHeader_1x16_P2.54mm_Vertical" (at 74.295 166.37 0)
+    (property "Footprint" "Connector_PinSocket_2.54mm:PinSocket_1x16_P2.54mm_Vertical" (at 74.295 166.37 0)
       (effects (font (size 1.27 1.27)) hide)
     )
@@
       (effects (font (size 1.27 1.27)) (justify left))
     )
-    (property "Footprint" "Connector_PinHeader_2.54mm:PinHeader_1x16_P2.54mm_Vertical" (at 42.545 167.005 0)
+    (property "Footprint" "Connector_PinSocket_2.54mm:PinSocket_1x16_P2.54mm_Vertical" (at 42.545 167.005 0)
       (effects (font (size 1.27 1.27)) hide)
     )
@@
     )
   )
+  (symbol (lib_id "power:PWR_FLAG") (at 23.495 153.67 0) (unit 1)
+    (in_bom yes) (on_board yes) (dnp no)
+    (property "Reference" "#FLG07" (at 23.495 151.765 0)
+      (effects (font (size 1.27 1.27)) hide)
+    )
+    (property "Value" "PWR_FLAG" (at 20.955 149.225 0)
+      (effects (font (size 1.27 1.27)))
+    )
+    (property "Footprint" "" (at 23.495 153.67 0)
+      (effects (font (size 1.27 1.27)) hide)
+    )
+    (property "Datasheet" "~" (at 23.495 153.67 0)
+      (effects (font (size 1.27 1.27)) hide)
+    )
+    (pin "1")
+    (instances
+      (project "Multi saturation module"
+        (path "/ec237045-c42e-41b5-9862-2d4c3f861897/c30b6378-be73-4bdd-8ae7-082c1f6babb1"
+          (reference "#FLG07") (unit 1)
+        )
+      )
+    )
+  )
   (symbol (lib_id "Device:R_Potentiometer_Trim") (at 142.875 99.06 0) (mirror x) (unit 1)
     (in_bom yes) (on_board yes) (dnp no)
@@
         (path "/ec237045-c42e-41b5-9862-2d4c3f861897/c30b6378-be73-4bdd-8ae7-082c1f6babb1"
           (reference "D2") (unit 1)
+        )
+      )
+    )
+  )
+  (symbol (lib_id "power:PWR_FLAG") (at 23.495 157.48 0) (unit 1)
+    (in_bom yes) (on_board yes) (dnp no)
+    (property "Reference" "#FLG08" (at 23.495 155.575 0)
+      (effects (font (size 1.27 1.27)) hide)
+    )
+    (property "Value" "PWR_FLAG" (at 22.86 159.385 0)
+      (effects (font (size 1.27 1.27)))
+    )
+    (property "Footprint" "" (at 23.495 157.48 0)
+      (effects (font (size 1.27 1.27)) hide)
+    )
+    (property "Datasheet" "~" (at 23.495 157.48 0)
+      (effects (font (size 1.27 1.27)) hide)
+    )
+    (pin "1")
+    (instances
+      (project "Multi saturation module"
+        (path "/ec237045-c42e-41b5-9862-2d4c3f861897/c30b6378-be73-4bdd-8ae7-082c1f6babb1"
+          (reference "#FLG08") (unit 1)
         )
       )
@@
         )
       )
+    )
+  )
+  (symbol (lib_id "power:PWR_FLAG") (at 37.465 149.225 0) (unit 1)
+    (in_bom yes) (on_board yes) (dnp no) (fields_autoplaced)
+    (property "Reference" "#FLG06" (at 37.465 147.32 0)
+      (effects (font (size 1.27 1.27)) hide)
+    )
+    (property "Value" "PWR_FLAG" (at 37.465 144.78 0)
+      (effects (font (size 1.27 1.27)))
+    )
+    (property "Footprint" "" (at 37.465 149.225 0)
+      (effects (font (size 1.27 1.27)) hide)
+    )
+    (property "Datasheet" "~" (at 37.465 149.225 0)
+      (effects (font (size 1.27 1.27)) hide)
+    )
+    (pin "1")
+    (instances
+      (project "Multi saturation module"
+        (path "/ec237045-c42e-41b5-9862-2d4c3f861897/c30b6378-be73-4bdd-8ae7-082c1f6babb1"
+          (reference "#FLG06") (unit 1)
+        )
+      )

Commit message: cleaned up project directory
Other:
- note added: "Bypass Switches"
- note added: "Gain trimmers"
- note added: "Global label format: Reference_Pin_Board"
- note added: "Indicator Leds"
- note added: "Jacks"
- note added: "Pots"
- moved on the sheet: D1, D2, D3, D5, D6, D?, J1, J3, J5, J?, R22, RV2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

Commit message: board and schematic update
Parts:
- added H3, H4: MountingHole, DIYSynthMNL:MountingHole_M3_Standoff_Pad, symbol Mechanical:MountingHole_Pad
- added H5, H6: MountingHole, DIYSynthMNL:MountingHole_M3_Euro, symbol Mechanical:MountingHole
Connections:
- net GND1: now also H3.1, H4.1
Changed lines of the file:
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@@
   (junction (at 108.585 81.28) (diameter 0) (color 0 0 0 0)
+  )
+  (junction (at 218.44 132.08) (diameter 0) (color 0 0 0 0)
   )
   (junction (at 151.13 57.785) (diameter 0) (color 0 0 0 0)
@@
     (stroke (width 0) (type default))
   )
+  (wire (pts (xy 222.885 132.08) (xy 218.44 132.08))
+    (stroke (width 0) (type default))
+  )
   (wire (pts (xy 188.595 130.81) (xy 187.325 130.81))
     (stroke (width 0) (type default))
@@
     (stroke (width 0) (type default))
   )
+  (wire (pts (xy 218.44 132.08) (xy 218.44 124.46))
+    (stroke (width 0) (type default))
+  )
   (wire (pts (xy 66.675 184.15) (xy 69.215 184.15))
+    (stroke (width 0) (type default))
+  )
+  (wire (pts (xy 218.44 124.46) (xy 222.885 124.46))
     (stroke (width 0) (type default))
   )
@@
         (path "/ec237045-c42e-41b5-9862-2d4c3f861897/c30b6378-be73-4bdd-8ae7-082c1f6babb1"
           (reference "#PWR016") (unit 1)
+        )
+      )
+    )
+  )
+  (symbol (lib_id "Mechanical:MountingHole") (at 247.015 120.65 0) (unit 1)
+    (in_bom yes) (on_board yes) (dnp no) (fields_autoplaced)
+    (property "Reference" "H5" (at 250.19 119.38 0)
+      (effects (font (size 1.27 1.27)) (justify left))
+    )
+    (property "Value" "MountingHole" (at 250.19 121.92 0)
+      (effects (font (size 1.27 1.27)) (justify left))
+    )
+    (property "Footprint" "DIYSynthMNL:MountingHole_M3_Euro" (at 247.015 120.65 0)
+      (effects (font (size 1.27 1.27)) hide)
+    )
+    (property "Datasheet" "~" (at 247.015 120.65 0)
+      (effects (font (size 1.27 1.27)) hide)
+    )
+    (instances
+      (project "Multi saturation module"
+        (path "/ec237045-c42e-41b5-9862-2d4c3f861897/c30b6378-be73-4bdd-8ae7-082c1f6babb1"
+          (reference "H5") (unit 1)
+        )
+      )
+    )
+  )
+  (symbol (lib_id "Mechanical:MountingHole") (at 247.015 127 0) (unit 1)
+    (in_bom yes) (on_board yes) (dnp no) (fields_autoplaced)
+    (property "Reference" "H6" (at 250.19 125.73 0)
+      (effects (font (size 1.27 1.27)) (justify left))
+    )
+    (property "Value" "MountingHole" (at 250.19 128.27 0)
+      (effects (font (size 1.27 1.27)) (justify left))
+    )
+    (property "Footprint" "DIYSynthMNL:MountingHole_M3_Euro" (at 247.015 127 0)
+      (effects (font (size 1.27 1.27)) hide)
+    )
+    (property "Datasheet" "~" (at 247.015 127 0)
+      (effects (font (size 1.27 1.27)) hide)
+    )
+    (instances
+      (project "Multi saturation module"
+        (path "/ec237045-c42e-41b5-9862-2d4c3f861897/c30b6378-be73-4bdd-8ae7-082c1f6babb1"
+          (reference "H6") (unit 1)
         )
       )
@@
     )
   )
+  (symbol (lib_id "Mechanical:MountingHole_Pad") (at 222.885 121.92 0) (unit 1)
+    (in_bom yes) (on_board yes) (dnp no) (fields_autoplaced)
+    (property "Reference" "H3" (at 226.06 119.38 0)
+      (effects (font (size 1.27 1.27)) (justify left))
+    )
+    (property "Value" "MountingHole" (at 226.06 121.92 0)
+      (effects (font (size 1.27 1.27)) (justify left))
+    )
+    (property "Footprint" "DIYSynthMNL:MountingHole_M3_Standoff_Pad" (at 222.885 121.92 0)
+      (effects (font (size 1.27 1.27)) hide)
+    )
+    (property "Datasheet" "~" (at 222.885 121.92 0)
+      (effects (font (size 1.27 1.27)) hide)
+    )
+    (pin "1")
+    (instances
+      (project "Multi saturation module"
+        (path "/ec237045-c42e-41b5-9862-2d4c3f861897/c30b6378-be73-4bdd-8ae7-082c1f6babb1"
+          (reference "H3") (unit 1)
+        )
+      )
+    )
+  )
   (symbol (lib_id "power:GND1") (at 151.13 78.74 0) (unit 1)
     (in_bom yes) (on_board yes) (dnp no) (fields_autoplaced)
@@
         (path "/ec237045-c42e-41b5-9862-2d4c3f861897/c30b6378-be73-4bdd-8ae7-082c1f6babb1"
           (reference "J5") (unit 1)
+        )
+      )
+    )
+  )
+  (symbol (lib_id "power:GND1") (at 218.44 132.08 0) (unit 1)
+    (in_bom yes) (on_board yes) (dnp no) (fields_autoplaced)
+    (property "Reference" "#PWR031" (at 218.44 138.43 0)
+      (effects (font (size 1.27 1.27)) hide)
+    )
+    (property "Value" "GND1" (at 218.44 136.525 0)
+      (effects (font (size 1.27 1.27)))
+    )
+    (property "Footprint" "" (at 218.44 132.08 0)
+      (effects (font (size 1.27 1.27)) hide)
+    )
+    (property "Datasheet" "" (at 218.44 132.08 0)
+      (effects (font (size 1.27 1.27)) hide)
+    )
+    (pin "1")
+    (instances
+      (project "Multi saturation module"
+        (path "/ec237045-c42e-41b5-9862-2d4c3f861897/c30b6378-be73-4bdd-8ae7-082c1f6babb1"
+          (reference "#PWR031") (unit 1)
         )
       )
@@
         )
       )
+    )
+  )
+  (symbol (lib_id "Mechanical:MountingHole_Pad") (at 222.885 129.54 0) (unit 1)
+    (in_bom yes) (on_board yes) (dnp no) (fields_autoplaced)
+    (property "Reference" "H4" (at 226.06 127 0)
+      (effects (font (size 1.27 1.27)) (justify left))
+    )
+    (property "Value" "MountingHole" (at 226.06 129.54 0)
+      (effects (font (size 1.27 1.27)) (justify left))
+    )
+    (property "Footprint" "DIYSynthMNL:MountingHole_M3_Standoff_Pad" (at 222.885 129.54 0)
+      (effects (font (size 1.27 1.27)) hide)
+    )
+    (property "Datasheet" "~" (at 222.885 129.54 0)
+      (effects (font (size 1.27 1.27)) hide)
+    )
+    (pin "1")
+    (instances
+      (project "Multi saturation module"
+        (path "/ec237045-c42e-41b5-9862-2d4c3f861897/c30b6378-be73-4bdd-8ae7-082c1f6babb1"
+          (reference "H4") (unit 1)
+        )
+      )
