File: Multiboard_Separate_Board_A/Multi saturation module_board_a.kicad_pcb (KiCad board)
At the start: 2 copper layers, 40 x 108.5 mm, 46 parts, among them J10 Board_A_1, J11 Board_A_2, J6 EuroPower_JST_3P, J7 EURO_PWR_16P, T1 TL016-R, U1 NE5532, U2 NE5532, U3 VTL5C, U4 NE5532, U5 NE5532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

Commit message: multiboard update, rounded tracks
Routing:
- net Board_0--12V: track 131.6 -> 127.0 mm
- net Board_0-+12V: track 148.1 -> 144.7 mm
- net Board_0-RV3_3: track 77.1 -> 74.6 mm
- net Board_0-Net-(U1B-+): track 24.1 -> 22.0 mm
- net Board_0-Dry: track 128.8 -> 126.8 mm
- net Board_0-Wet: track 73.4 -> 71.4 mm
- net Board_0-Mix_audio_out: track 39.0 -> 37.1 mm
- net Board_0-Net-(R16-Pad2): track 16.0 -> 14.3 mm
- net Board_0-SW1_4: track 47.1 -> 45.4 mm
- net Board_0-RV2_3: track 81.0 -> 79.3 mm
- net Board_0-Net-(U5B--): track 29.0 -> 27.2 mm
- net Board_0-SW2_2: track 37.4 -> 36.0 mm
- net Board_0-Audio_in: track 33.3 -> 32.0 mm
- net Board_0-Net-(R15-Pad1): track 22.0 -> 20.7 mm
- net Board_0-Clipping_diodes: track 81.3 -> 80.1 mm
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Other:
- board text added: "+12V"
- board text added: "-12V"
- board text added: "GND"
