File: Multiboard_Separate_Board_B/Multi saturation module_board_b.kicad_pcb (KiCad board)
At the start: 2 copper layers, 40 x 108.5 mm, 23 parts, among them J1 Mix_audio_out, J2 Audio_in, J4 Mix_CV_in, J5 Wet_audio_out, J8 Board_B_1, J9 Board_B_2, SW1 Clipping, SW2 Xformer_bypass, SW3 Opto_bypass

Commit message: multiboard update, rounded tracks
Routing:
- net Board_0-SW1_1_B: track 53.5 -> 50.5 mm
- net Board_0-RV2_3_B: track 61.2 -> 59.3 mm
- net Board_0-SW1_2_B: track 43.2 -> 41.3 mm
- net Board_0-Mix_CV_in_B: track 67.1 -> 65.2 mm
- net Board_0-RV1_2_B: track 39.9 -> 38.1 mm
- net Board_0-Mix_audio_out_B: track 94.8 -> 93.1 mm
- net Board_0-RV4_3_B: track 29.7 -> 28.1 mm
- net Board_0-Wet_B: track 69.7 -> 68.5 mm
- net Board_0-SW2_2_B: track 33.2 -> 32.0 mm
- net Board_0-Clipping_diodes_B: track 60.3 -> 59.1 mm
- net Board_0-+12VA: track 68.7 -> 67.6 mm
- net Board_0-SW1_4_B: track 38.4 -> 37.3 mm
- net Board_0-SW2_1_B: track 28.1 -> 27.0 mm
- net Board_0-D4_-_B: track 47.9 -> 46.9 mm
- net Board_0-RV3_3_B: track 48.6 -> 47.7 mm
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Other:
- board text added: "Multi Saturation Rev 0.1"
